File: Dev Kit/SOFTWEAR_microbit2.sch (EAGLE design)
At the start: 11 parts, among them J1 EDGE-80PTH-RA, J2 M22PTH, J3 QWIIC_RIGHT_ANGLE, X1 SM03B-SRSS-TB, X2 SM03B-SRSS-TB, X3 SM03B-SRSS-TB

Commit message: updated design
Parts:
- added X4, X5, X6: SM03B-SRSS-TB, con-JST SH (1):SM03B-SRSS-TB
- J2: value M22PTH -> (none); device local_lib:M22PTH -> SparkFun-Connectors:JST_2MM_MALE
Connections:
- removed net 12: J1.A23, J2.16
- removed net 16: J1.A15, J2.20
- removed net 8: J1.A27, J2.12
- removed net AUD: J1.A40, J2.7, X2.1
- removed net NEO: J1.A28, J1.A29, J1.A30, J1.A31, J2.5, X3.1
- removed net VIBE: J1.A19, J1.A20, J1.A21, J1.A22, J2.6, X1.1
- new net 1: J1.A28, J1.A29, J1.A30, J1.A31, X1.1
- new net 2: J1.A19, J1.A20, J1.A21, J1.A22, X3.1
- new net 3: J1.A40
- new net NEO1: J1.A27, X4.1
- new net NEO2: J1.A23, X5.1
- new net NEO3: J1.A15, X6.1
- new net V_BATT: J2.+, X4.3, X5.3, X6.3
- net 0: now also X2.1; no longer J2.4
- net 10: no longer J2.14
- net 11: no longer J2.15
- net 13: no longer J2.17
- net 14: no longer J2.18
- net 15: no longer J2.19
- net 3.3V: no longer J2.3
- net 4: no longer J2.8
- net 5: no longer J2.9
- net 6: no longer J2.10
- net 7: no longer J2.11
- net 9: no longer J2.13
- net GND: now also J2.-, X4.2, X5.2, X6.2; no longer J2.1, J2.2
- net SCL: no longer J2.21
- net SDA: no longer J2.22
